File: catlamp.kicad_pcb (KiCad board)
At the start: 2 copper layers, 57.8 x 57.8 mm, 43 parts, among them J1 Bat, J2 Charger, J3 LED, J4 TTP4, J5 TTP5, Q1 AO3401, Q2 BSS138, U1 TP4056, U2 DW01, U3 FS8205A, U4 ESP32, U5 MCP1700T, U7 74AUP1G08, U8 TPS61023DRLR

Commit message: New design using the BQ24075RGT Battery management IC
Parts:
- removed C1: 0.1uF, Capacitor_SMD:C_0805_2012Metric_Pad1.18x1.45mm_HandSolder
- removed C2, C7: 10uF, Capacitor_SMD:C_0805_2012Metric_Pad1.18x1.45mm_HandSolder
- removed C3, C6: 100nF, Capacitor_SMD:C_0805_2012Metric_Pad1.18x1.45mm_HandSolder
- removed C4: 1000uF, Capacitor_SMD:CP_Elec_10x10
- removed C5: 100uF, Capacitor_SMD:CP_Elec_5x5.4
- removed C8, C9: 22uF, Capacitor_SMD:C_0805_2012Metric_Pad1.18x1.45mm_HandSolder
- removed D3: SS14, Diode_SMD:D_SMA_Handsoldering
- removed Q1: AO3401, Package_TO_SOT_SMD:TSOT-23_HandSoldering
- removed R1, R2, R4: 1k, Resistor_SMD:R_0805_2012Metric_Pad1.20x1.40mm_HandSolder
- removed R10, R9: 10k, Resistor_SMD:R_0805_2012Metric_Pad1.20x1.40mm_HandSolder
- removed R3: 1.2k, Resistor_SMD:R_0805_2012Metric_Pad1.20x1.40mm_HandSolder
- removed R5, R7, R8: 100k, Resistor_SMD:R_0805_2012Metric_Pad1.20x1.40mm_HandSolder
- removed R6: 100, Resistor_SMD:R_0805_2012Metric_Pad1.20x1.40mm_HandSolder
- removed U7: 74AUP1G08, Package_TO_SOT_SMD:SOT-23-5_HandSoldering
- removed U8: TPS61023DRLR, extern:SOT563-ORI
- added C11: 1uF, Capacitor_SMD:C_0805_2012Metric_Pad1.18x1.45mm_HandSolder, F.Cu at (138.3, 118.2)
- added C12: 10uF, Capacitor_SMD:C_0805_2012Metric_Pad1.18x1.45mm_HandSolder, F.Cu at (142.8, 122.8)
- added C13: 10uF, Capacitor_SMD:C_0805_2012Metric_Pad1.18x1.45mm_HandSolder, F.Cu at (143.8, 115.0)
- added C21: 10uF, Capacitor_SMD:C_0805_2012Metric_Pad1.18x1.45mm_HandSolder, F.Cu at (157.3, 107.0)
- added C22: 22uF, Capacitor_SMD:C_0805_2012Metric_Pad1.18x1.45mm_HandSolder, F.Cu at (163.4, 106.0)
- added C23: 22uF, Capacitor_SMD:C_0805_2012Metric_Pad1.18x1.45mm_HandSolder, F.Cu at (165.4, 106.0)
- added C24: 220pF, Capacitor_SMD:C_0805_2012Metric_Pad1.18x1.45mm_HandSolder, F.Cu at (160.5, 103.8)
- added C31: 1uF, Capacitor_SMD:C_0805_2012Metric_Pad1.18x1.45mm_HandSolder, F.Cu at (160.3, 87.0)
- added C32: 1uF, Capacitor_SMD:C_0805_2012Metric_Pad1.18x1.45mm_HandSolder, F.Cu at (160.2, 96.2)
- added C41: 47uF, Capacitor_SMD:C_0805_2012Metric_Pad1.18x1.45mm_HandSolder, F.Cu at (158.8, 80.5)
- added C42: 100nF, Capacitor_SMD:C_0805_2012Metric_Pad1.18x1.45mm_HandSolder, F.Cu at (168.2, 94.3)
- added C43: 100nF, Capacitor_SMD:C_0805_2012Metric_Pad1.18x1.45mm_HandSolder, F.Cu at (129.4, 95.7)
- added C44: 100nF, Capacitor_SMD:C_0805_2012Metric_Pad1.18x1.45mm_HandSolder, F.Cu at (135.5, 87.7)
- added H1: MountingHole, MountingHole:MountingHole_2.2mm_M2, F.Cu at (2.48, 2.48)
- added H2: MountingHole, MountingHole:MountingHole_2.2mm_M2, F.Cu at (2.48, 8.43)
- added H3: MountingHole, MountingHole:MountingHole_2.2mm_M2, F.Cu at (2.48, 14.4)
- added R14: 51k, Resistor_SMD:R_0805_2012Metric_Pad1.20x1.40mm_HandSolder, F.Cu at (138.3, 120.2)
- added R15: 1.2k, Resistor_SMD:R_0805_2012Metric_Pad1.20x1.40mm_HandSolder, F.Cu at (141.3, 115.0)
- added R16: 1k, Resistor_SMD:R_0805_2012Metric_Pad1.20x1.40mm_HandSolder, F.Cu at (138.6, 123.2)
- added R21: 51k, Resistor_SMD:R_0805_2012Metric_Pad1.20x1.40mm_HandSolder, F.Cu at (162.9, 100.0)
- added R22: 680k, Resistor_SMD:R_0805_2012Metric_Pad1.20x1.40mm_HandSolder, F.Cu at (159.8, 101.0)
- added R23: 100k, Resistor_SMD:R_0805_2012Metric_Pad1.20x1.40mm_HandSolder, F.Cu at (157.4, 101.0)
- added R41: 100k, Resistor_SMD:R_0805_2012Metric_Pad1.20x1.40mm_HandSolder, F.Cu at (145.0, 100.8)
- added R42: 100k, Resistor_SMD:R_0805_2012Metric_Pad1.20x1.40mm_HandSolder, F.Cu at (150.4, 100.8)
- added R43: 10k, Resistor_SMD:R_0805_2012Metric_Pad1.20x1.40mm_HandSolder, F.Cu at (164.1, 90.5)
- added R44: 10k, Resistor_SMD:R_0805_2012Metric_Pad1.20x1.40mm_HandSolder, F.Cu at (168.2, 103.0)
- H1: renamed from REF1; value MountingHole_2.2mm_M2 -> Conn_01x01_MountingPin
- H2: renamed from REF2; value MountingHole_2.2mm_M2 -> Conn_01x01_MountingPin
- H3: renamed from REF3; value MountingHole_2.2mm_M2 -> Conn_01x01_MountingPin
- R11: value 680k -> 10k
- R12: value 51k -> 1.5k
- R13: value 10k -> 1.5k
- U1: value TP4056 -> BQ24075RGT; footprint Package_SO:SOIC-8-1EP_3.9x4.9mm_P1.27mm_EP2.29x3mm -> Package_DFN_QFN:VQFN-16-1EP_3x3mm_P0.5mm_EP1.6x1.6mm
- U2: value DW01 -> TPS61023DRLR; footprint Package_TO_SOT_SMD:SOT-23-6_Handsoldering -> extern:SOT563-ORI
- U3: value FS8205A -> MCP1700T; footprint Package_TO_SOT_SMD:SOT-23-6_Handsoldering -> Package_TO_SOT_SMD:SOT-23_Handsoldering
- U5: value MCP1700T -> 74AUP1G08; footprint Package_TO_SOT_SMD:SOT-23_Handsoldering -> Package_TO_SOT_SMD:SOT-23-5_HandSoldering
- moved U3 36.1 mm to (160.3, 91.0), turned to -90 degrees
- moved R13 35.1 mm to (126.5, 102.0), turned to 180 degrees
- moved R12 29.8 mm to (126.5, 99.0), turned to 180 degrees
- moved R11 29.1 mm to (136.4, 123.2), turned to -90 degrees
- moved U2 21.8 mm to (160.9, 106.0), turned to -90 degrees
- moved L1 13.5 mm to (157.8, 111.8)
- moved U1 10.9 mm to (143.8, 119.4), turned to 90 degrees
- moved U5 3.62 mm to (134.1, 91.7), turned to 0 degrees
- moved Q2 3.40 mm to (165.0, 95.4), turned to -90 degrees
- turned D1 to 0 degrees
- turned D2 to 0 degrees
Connections:
- D1 pad 2: VIN -> Net-(D1-A)
- D2 pad 2: VIN -> Net-(D2-A)
- J1 pad 1: BAT- -> GND
- J2 pad 2: VIN -> Net-(J2-Pin_2)
- L1 pad 2: Net-(U8-SW) -> Net-(U2-SW)
- R11 pad 1: Net-(R11-Pad1) -> Net-(U1-TS)
- R11 pad 2: Net-(U8-FB) -> GND
- R12 pad 1: 5V -> VOUT
- R12 pad 2: Net-(R11-Pad1) -> Net-(D1-A)
- R13 pad 1: VIN -> VOUT
- R13 pad 2: GND -> Net-(D2-A)
- U1 pad 1: GND -> Net-(U1-TS)
- U1 pad 2: Net-(U1-PROG) -> BAT+
- U1 pad 3: GND -> BAT+
- U1 pad 4: VIN -> GND
- U1 pad 5: BAT+ -> VOUT
- U1 pad 6: Net-(U1-~{STDBY}) -> GND
- U1 pad 7: Net-(U1-~{CHRG}) -> Net-(D2-K)
- U1 pad 8: VIN -> GND
- U1 pad 9: GND -> Net-(D1-K)
- U2 pad 1: /G1 -> Net-(U2-FB)
- U2 pad 2: Net-(U2-CS) -> EN
- U2 pad 3: /G2 -> VOUT
- U2 pad 4: unconnected-(U2-TD-Pad4) -> GND
- U2 pad 5: Net-(U2-VCC) -> Net-(U2-SW)
- U2 pad 6: BAT- -> 5V
- U3 pad 1: BAT- -> GND
- U3 pad 2: unconnected-(U3-D1D2-Pad2) -> 3.3V
- U3 pad 3: GND -> VOUT
- U5 pad 1: GND -> IO5
- U5 pad 2: 3.3V -> IO4
- U5 pad 3: VOUT -> GND
Routing:
- net VIN: track 77.8 -> 0.00 mm, vias 2 -> 0
- net BAT+: track 75.7 -> 31.2 mm, vias 6 -> 2
- net BAT-: track 34.9 -> 0.00 mm, vias 2 -> 0
- net 5V: track 36.6 -> 3.32 mm
- net Net-(J2-Pin_2): track 0.00 -> 31.5 mm, vias 0 -> 2
- net Net-(D2-K): track 2.88 -> 33.9 mm
- net Net-(D1-K): track 2.88 -> 32.8 mm
- net Net-(U2-CS): track 22.7 -> 0.00 mm, vias 2 -> 0
- net Net-(U1-~{CHRG}): track 21.7 -> 0.00 mm, vias 2 -> 0
- net Net-(U2-VCC): track 21.5 -> 0.00 mm, vias 2 -> 0
- net Net-(U1-~{STDBY}): track 19.6 -> 0.00 mm, vias 2 -> 0
- net Net-(U8-FB): track 19.0 -> 0.00 mm, vias 2 -> 0
- net IO5: track 39.4 -> 24.7 mm, vias 2 -> 0
- net 3.3V: track 102.1 -> 88.6 mm, vias 2 -> 3
- net GND: track 2.36 -> 14.7 mm, vias 178 -> 297
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- added copper zone on F.Cu, net 5V
- added copper zone on F.Cu, net BAT+
- added copper zone on F.Cu, net Net-(J2-Pin_2)
- added copper zone on F.Cu, net Net-(U2-FB)
- added copper zone on F.Cu, net VOUT
