File: catlamp.kicad_sch (KiCad schematic)
At the start: 41 parts, among them J1 Bat, J2 Charger, J3 LED, J4 TTP4, J5 TTP5, Q1 AO3401, Q2 BSS138, SW1 SW_SPST, U1 TP4056, U2 DW01, U3 FS8205A, U4 ESP32, U5 MCP1700T, U7 74AUP1G08, U8 TPS61023DRLR

Commit message: New design using the BQ24075RGT Battery management IC
Parts:
- removed C1: 0.1uF, Capacitor_SMD:C_0805_2012Metric_Pad1.18x1.45mm_HandSolder, symbol Device:C
- removed C2: 10uF, Capacitor_SMD:C_0805_2012Metric_Pad1.18x1.45mm_HandSolder, symbol Device:C
- removed C3: 100nF, Capacitor_SMD:C_0805_2012Metric_Pad1.18x1.45mm_HandSolder, symbol Device:C
- removed C4: 1000uF, Capacitor_SMD:CP_Elec_10x10, symbol Device:C_Polarized
- removed C5: 100uF, Capacitor_SMD:CP_Elec_5x5.4, symbol Device:C_Polarized
- removed D3: SS14, Diode_SMD:D_SMA_Handsoldering, symbol Diode:SS14
- removed Q1: AO3401, Package_TO_SOT_SMD:TSOT-23_HandSoldering, symbol extern:AO3401
- removed R1, R2, R4: 1k, Resistor_SMD:R_0805_2012Metric_Pad1.20x1.40mm_HandSolder, symbol Device:R
- removed R3: 1.2k, Resistor_SMD:R_0805_2012Metric_Pad1.20x1.40mm_HandSolder, symbol Device:R
- removed R6: 100, Resistor_SMD:R_0805_2012Metric_Pad1.20x1.40mm_HandSolder, symbol Device:R
- removed SW1: SW_SPST, symbol Switch:SW_SPST
- removed U1: TP4056, Package_SO:SOIC-8-1EP_3.9x4.9mm_P1.27mm_EP2.29x3mm, symbol tp4056:TP4056
- removed U2: DW01, Package_TO_SOT_SMD:SOT-23-6_Handsoldering, symbol dw01:DW01
- removed U3: FS8205A, Package_TO_SOT_SMD:SOT-23-6_Handsoldering, symbol fs8205:FS8205A
- added C11, C31, C32: 1uF, Capacitor_SMD:C_0805_2012Metric_Pad1.18x1.45mm_HandSolder, symbol Device:C
- added C12, C13: 10uF, Capacitor_SMD:C_0805_2012Metric_Pad1.18x1.45mm_HandSolder, symbol Device:C
- added C24: 220pF, Capacitor_SMD:C_0805_2012Metric_Pad1.18x1.45mm_HandSolder, symbol Device:C
- added C42, C43, C44: 100nF, Capacitor_SMD:C_0805_2012Metric_Pad1.18x1.45mm_HandSolder, symbol Device:C
- added H1, H2, H3: MountingHole, MountingHole:MountingHole_2.2mm_M2, symbol Mechanical:MountingHole
- added R11: 10k, Resistor_SMD:R_0805_2012Metric_Pad1.20x1.40mm_HandSolder, symbol Device:R
- added R12: 1.5k, Resistor_SMD:R_0805_2012Metric_Pad1.20x1.40mm_HandSolder, symbol Device:R
- added R14: 51k, Resistor_SMD:R_0805_2012Metric_Pad1.20x1.40mm_HandSolder, symbol Device:R
- added R15: 1.2k, Resistor_SMD:R_0805_2012Metric_Pad1.20x1.40mm_HandSolder, symbol Device:R
- added R16: 1k, Resistor_SMD:R_0805_2012Metric_Pad1.20x1.40mm_HandSolder, symbol Device:R
- added U1: BQ24075RGT, Package_DFN_QFN:VQFN-16-1EP_3x3mm_P0.5mm_EP1.6x1.6mm, symbol Battery_Management:BQ24075RGT
- C41: renamed from C6; value 100nF -> 47uF
- R13: value 10k -> 1.5k
- renumbered C7 to C21, C8 to C22, C9 to C23, R12 to R21, R11 to R22, R5 to R23, R7 to R41, R8 to R42, R9 to R43, R10 to R44, U8 to U2, U5 to U3, U7 to U5
Connections:
- net BAT- is gone; now on net GND: J1.1 (Pin_1)
- net 3.3V: now also C31.1, C42.2, C43.2, C44.2
- net 5V: now also C24.1
- net BAT+: now also J1.2 (Pin_2), C12.2, U1.2 (BAT), U1.3 (BAT)
- net GND: now also C11.1, C12.1, C13.1, C31.2, C32.2, C42.1, C43.1, C44.1, R11.2, R14.1, R15.1, R16.1, U1.15 (SYSOFF), U1.17 (VSS), U1.4 (~{CE}), U1.6 (EN1), U1.8 (VSS); no longer R13.2
- net VOUT: now also R13.1, C13.2, C32.1, R12.1, U1.10 (OUT), U1.11 (OUT), U1.5 (EN2)
- net at D1.1 (K): now also U1.9 (~{CHG})
- net at D2.1 (K): now also U1.7 (~{PGOOD})
- net at R22.2, R23.2, U2.1 (FB): now also C24.2
- removed net VIN: D1.2 (A), D2.2 (A), J2.2 (Pin_2), R13.1
- new net: D1.2 (A), R12.2
- new net: R11.1, U1.1 (TS)
- new net: R15.2, U1.12 (ILIM)
- new net: C11.2, J2.2 (Pin_2), U1.13 (IN)
- new net: R14.2, U1.14 (TMR)
- new net: R16.2, U1.16 (ISET)
- new net: D2.2 (A), R13.2
- no-connect marks 3 -> 0
Other:
- note removed: "Elko"
- note removed: "Ground Temp disables Temperature sensor"
- note removed: "R3 set chargin current 1.2k = 1000 ma"
- moved on the sheet: C21, C22, C23, J3, J4, J5, L1, Q2, R21, R22, R23, R41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
